File: RF_Defence.kicad_pcb (KiCad board)
At the start: 2 copper layers, 43.2 x 17.8 mm, 37 parts, among them J1 Analog, J2 Digital, U1 LM358_DFN, U2 LM358, U3 LM358, U4 LM358_DFN, U5 LM358, U6 LM358_DFN

Commit message: Add files via upload
Routing:
- net +3V3: track 39.6 -> 176.9 mm
- net /D8: track 0.00 -> 83.6 mm
- net /D7: track 0.00 -> 76.2 mm
- net /A1: track 5.43 -> 66.7 mm
- net GND: track 208.2 -> 259.6 mm
- net Net-(D1-A): track 46.8 -> 96.9 mm
- net Net-(D2-A): track 36.0 -> 60.8 mm
- net /~{RESET}: track 0.00 -> 15.2 mm
- net (no net): track 76.2 -> 73.3 mm
Other:
- board size 43.2 x 17.8 mm -> 91.6 x 74.2 mm
